File: Slim Keyboard.kicad_sch (KiCad schematic)
At the start: 4 parts

Commit message: Updated Footprints
Parts:
- rBT1, rBT2, rBT3, rBT4: footprint kbd_local:Breakaway_Tabs -> Panelization:BreakLine_9h_D0.5mm_P0.85mm
Changed lines of the file:
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@@
 			)
 		)
-		(property "Footprint" "kbd_local:Breakaway_Tabs"
+		(property "Footprint" "Panelization:BreakLine_9h_D0.5mm_P0.85mm"
 			(at 19.05 190.5 0)
 			(effects
@@
 			)
 		)
-		(property "Footprint" "kbd_local:Breakaway_Tabs"
+		(property "Footprint" "Panelization:BreakLine_9h_D0.5mm_P0.85mm"
 			(at 19.05 184.15 0)
 			(effects
@@
 			)
 		)
-		(property "Footprint" "kbd_local:Breakaway_Tabs"
+		(property "Footprint" "Panelization:BreakLine_9h_D0.5mm_P0.85mm"
 			(at 19.05 171.45 0)
 			(effects
@@
 			)
 		)
-		(property "Footprint" "kbd_local:Breakaway_Tabs"
+		(property "Footprint" "Panelization:BreakLine_9h_D0.5mm_P0.85mm"
 			(at 19.05 177.8 0)
 			(effects

Commit message: Started PCB design
Parts:
- removed rBT1, rBT2, rBT3, rBT4: Breakaway Tabs, Panelization:BreakLine_9h_D0.5mm_P0.85mm, symbol Mechanical:MountingHole
