File: alt_leds.kicad_sch (KiCad schematic)
At the start: 23 parts

Commit message: Connected GPIO
Connections:
- no-connect marks 18 -> 46
Changed lines of the file:
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@@
+	)
+	(no_connect
+		(at 101.6 105.41)
+	)
+	(no_connect
+		(at 49.53 74.93)
+	)
+	(no_connect
+		(at 113.03 83.82)
+	)
+	(no_connect
+		(at 127 105.41)
+	)
+	(no_connect
+		(at 80.01 83.82)
 	)
 	(no_connect
 		(at 80.01 63.5)
+	)
+	(no_connect
+		(at 113.03 73.66)
+	)
+	(no_connect
+		(at 107.95 63.5)
+	)
+	(no_connect
+		(at 93.98 105.41)
 	)
 	(no_connect
@@
 	)
 	(no_connect
+		(at 87.63 83.82)
+	)
+	(no_connect
 		(at 87.63 73.66)
 	)
@@
 	)
 	(no_connect
+		(at 114.3 125.73)
+	)
+	(no_connect
+		(at 41.91 106.68)
+	)
+	(no_connect
+		(at 49.53 118.11)
+	)
+	(no_connect
 		(at 86.36 35.56)
 	)
 	(no_connect
+		(at 41.91 118.11)
+	)
+	(no_connect
 		(at 86.36 46.99)
+	)
+	(no_connect
+		(at 49.53 63.5)
+	)
+	(no_connect
+		(at 134.62 105.41)
+	)
+	(no_connect
+		(at 120.65 73.66)
+	)
+	(no_connect
+		(at 73.66 125.73)
 	)
 	(no_connect
@@
 	)
 	(no_connect
+		(at 113.03 63.5)
+	)
+	(no_connect
+		(at 41.91 74.93)
+	)
+	(no_connect
+		(at 100.33 63.5)
+	)
+	(no_connect
+		(at 114.3 105.41)
+	)
+	(no_connect
+		(at 41.91 63.5)
+	)
+	(no_connect
 		(at 68.58 105.41)
+	)
+	(no_connect
+		(at 81.28 125.73)
 	)
 	(no_connect
@@
 	)
 	(no_connect
+		(at 49.53 106.68)
+	)
+	(no_connect
+		(at 120.65 83.82)
+	)
+	(no_connect
 		(at 81.28 105.41)
 	)
 	(no_connect
 		(at 73.66 35.56)
+	)
+	(no_connect
+		(at 120.65 63.5)
 	)
 	(no_connect
@@
 	)
 	(no_connect
+		(at 106.68 105.41)
+	)
+	(no_connect
+		(at 106.68 125.73)
+	)
+	(no_connect
